File: nav_system.kicad_sch (KiCad schematic)
At the start: 16 parts, among them J1 GPS MODULE, J2 MPU6050, J3 SIM76003-L1C, J4 ESP32-CAM, J5 SW-420, J6 Conn_01x02_Socket, J7 SW-420 TOGGLE, J8 RGB, J9 RGB_GROUND, SW1 SW_SPDT

Commit message: Trying to add 3d model
Parts:
- removed D1, D2, D3: LED, symbol Device:LED
- removed J7: SW-420 TOGGLE, symbol Connector:Conn_01x03_Socket
- removed SW1: SW_SPDT, symbol Switch:SW_SPDT
- added C1: C_Polarized, Capacitor_THT:CP_Radial_D10.0mm_P3.50mm, symbol Device:C_Polarized
- added J10: SW-420, Connector_JST:JST_XH_B3B-XH-A_1x03_P2.50mm_Vertical, symbol Connector:Conn_01x03_Socket
- added U1: (no value), SHIELD:ESP32_38, symbol SHIELD:ESP32_38
- J1: footprint (none) -> Connector_PinSocket_2.54mm:PinSocket_1x04_P2.54mm_Vertical
- J2: footprint (none) -> Connector_PinSocket_2.54mm:PinSocket_1x08_P2.54mm_Vertical
- J3: footprint (none) -> Connector_PinSocket_2.54mm:PinSocket_1x07_P2.54mm_Vertical
- J4: footprint (none) -> Connector_JST:JST_XH_B2B-XH-A_1x02_P2.50mm_Vertical
- J5, J8, J9: footprint (none) -> Connector_JST:JST_XH_B3B-XH-A_1x03_P2.50mm_Vertical
- J6: value Conn_01x02_Socket -> MAIN POWER; footprint (none) -> Connector_JST:JST_XH_B2B-XH-A_1x02_P2.50mm_Vertical
- R1, R2, R3: footprint (none) -> Resistor_THT:R_Axial_DIN0204_L3.6mm_D1.6mm_P5.08mm_Horizontal
Connections:
- net BLUE: now also U1.10 (G26); no longer J8.2 (Pin_2)
- net DO: now also U1.5 (G34)
- net GND: now also J6.1 (Pin_1), J9.1 (Pin_1), J9.2 (Pin_2), J9.3 (Pin_3), C1.2, J10.1 (Pin_1), U1.14 (GND), U1.32 (GND), U1.38 (GND)
- net GREEN: now also U1.9 (G25); no longer J8.3 (Pin_3)
- net PWRKEY: now also U1.30 (G18)
- net RED: now also U1.11 (G27); no longer J8.1 (Pin_1)
- net RX: now also U1.7 (G32)
- net RXD: now also U1.28 (G17)
- net SCL: now also U1.37 (G23)
- net SDA: now also U1.33 (G21)
- net TX: now also U1.8 (G33)
- net TXD: now also U1.27 (G16)
- net VCC: now also J6.2 (Pin_2), C1.1, U1.19 (V5); no longer J2.8 (Pin_8)
- net at R2.1: now also J8.2 (Pin_2)
- net at R3.1: now also J8.3 (Pin_3)
- net at R1.1: now also J8.1 (Pin_1)
- new net +3.3V: J10.3 (Pin_3), J2.8 (Pin_8), U1.1 (3V3)
- new net g5: J10.2 (Pin_2), U1.29 (G5)
- no-connect marks 0 -> 27
Other:
- note added: "ESP32 38 PINS"
- note added: "LED INDICATORS"
- note added: "MODULES"
- note added: "SWITCHES"
- moved on the sheet: J4, J5, J6, J9, R1, R2, R3

Commit message: Nav_system.2.0
Parts:
- removed J1: GPS MODULE, Connector_PinSocket_2.54mm:PinSocket_1x04_P2.54mm_Vertical, symbol Connector:Conn_01x04_Socket
- added J1: gps module, Connector_PinHeader_2.54mm:PinHeader_1x05_P2.54mm_Vertical, symbol Connector:Conn_01x05_Socket
- added J11: MAIN P SWITCH, Connector_JST:JST_XH_B2B-XH-A_1x02_P2.50mm_Vertical, symbol Connector:Conn_01x02_Socket
- added J7: DC FAN, Connector_JST:JST_XH_B2B-XH-A_1x02_P2.50mm_Vertical, symbol Connector:Conn_01x02_Socket
- J10: value SW-420 -> toggle
- J5: footprint Connector_JST:JST_XH_B3B-XH-A_1x03_P2.50mm_Vertical -> Connector_PinSocket_2.54mm:PinSocket_1x03_P2.54mm_Vertical
Connections:
- net DO: now also J5.1 (Pin_1); no longer J5.2 (Pin_2)
- net GND: now also J5.2 (Pin_2), J1.4 (Pin_4), J7.2 (Pin_2); no longer J5.1 (Pin_1)
- net RX: now also J1.2 (Pin_2)
- net RXD: now also J3.3 (Pin_3); no longer J3.2 (Pin_2)
- net TX: now also J1.3 (Pin_3)
- net TXD: now also J3.2 (Pin_2); no longer J3.3 (Pin_3)
- net VCC: now also J1.5 (Pin_5), J11.2 (Pin_2), J7.1 (Pin_1); no longer J6.2 (Pin_2)
- new net: J11.1 (Pin_1), J6.2 (Pin_2)
Other:
- moved on the sheet: J6

Commit message: modify plot files
Other:
- moved on the sheet: C1, J4
Changed lines of the file:
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@@
 	)
 	(junction
-		(at 203.2 39.37)
+		(at 196.85 39.37)
 		(diameter 0)
 		(color 0 0 0 0)
@@
 	)
 	(junction
-		(at 203.2 31.75)
+		(at 196.85 31.75)
 		(diameter 0)
 		(color 0 0 0 0)
@@
 	(wire
 		(pts
-			(xy 203.2 31.75) (xy 203.2 34.29)
+			(xy 196.85 31.75) (xy 196.85 34.29)
 		)
 		(stroke
@@
 	(wire
 		(pts
-			(xy 199.39 34.29) (xy 203.2 34.29)
+			(xy 193.04 34.29) (xy 196.85 34.29)
 		)
 		(stroke
@@
 	(wire
 		(pts
-			(xy 203.2 31.75) (xy 209.55 31.75)
+			(xy 196.85 31.75) (xy 203.2 31.75)
 		)
 		(stroke
@@
 	(wire
 		(pts
-			(xy 203.2 36.83) (xy 203.2 39.37)
+			(xy 196.85 36.83) (xy 196.85 39.37)
 		)
 		(stroke
@@
 	(wire
 		(pts
-			(xy 199.39 36.83) (xy 203.2 36.83)
+			(xy 193.04 36.83) (xy 196.85 36.83)
 		)
 		(stroke
@@
 	(wire
 		(pts
-			(xy 209.55 39.37) (xy 203.2 39.37)
+			(xy 203.2 39.37) (xy 196.85 39.37)
 		)
 		(stroke
@@
 	(wire
 		(pts
-			(xy 203.2 30.48) (xy 203.2 31.75)
+			(xy 196.85 30.48) (xy 196.85 31.75)
 		)
 		(stroke
@@
 	(symbol
 		(lib_id "power:VCC")
-		(at 203.2 30.48 0)
+		(at 196.85 30.48 0)
 		(unit 1)
 		(body_style 1)
@@
 		(fields_autoplaced yes)
 		(property "Reference" "#PWR03"
-			(at 203.2 34.29 0)
+			(at 196.85 34.29 0)
 			(hide yes)
 			(show_name no)
@@
 		)
 		(property "Value" "VCC"
-			(at 203.2 25.4 0)
+			(at 196.85 25.4 0)
 			(show_name no)
 			(do_not_autoplace no)
@@
 		)
 		(property "Footprint" ""
-			(at 203.2 30.48 0)
+			(at 196.85 30.48 0)
 			(hide yes)
 			(show_name no)
@@
 		)
 		(property "Datasheet" ""
-			(at 203.2 30.48 0)
+			(at 196.85 30.48 0)
 			(hide yes)
 			(show_name no)
@@
 		)
 		(property "Description" "Power symbol creates a global label with name \"VCC\""
-			(at 203.2 30.48 0)
+			(at 196.85 30.48 0)
 			(hide yes)
 			(show_name no)
@@
 	(symbol
 		(lib_id "Connector:Conn_01x02_Socket")
-		(at 194.31 36.83 180)
+		(at 187.96 36.83 180)
 		(unit 1)
 		(body_style 1)
@@
 		(fields_autoplaced yes)
 		(property "Reference" "J4"
-			(at 194.945 29.21 0)
+			(at 188.595 29.21 0)
 			(show_name no)
 			(do_not_autoplace no)
@@
 		)
 		(property "Value" "ESP32-CAM"
-			(at 194.945 31.75 0)
+			(at 188.595 31.75 0)
 			(show_name no)
 			(do_not_autoplace no)
@@
 		)
 		(property "Footprint" "Connector_JST:JST_XH_B2B-XH-A_1x02_P2.50mm_Vertical"
-			(at 194.31 36.83 0)
+			(at 187.96 36.83 0)
 			(hide yes)
 			(show_name no)
@@
 		)
 		(property "Datasheet" ""
-			(at 194.31 36.83 0)
+			(at 187.96 36.83 0)
 			(hide yes)
 			(show_name no)
@@
 		)
 		(property "Description" "Generic connector, single row, 01x02, script generated"
-			(at 194.31 36.83 0)
+			(at 187.96 36.83 0)
 			(hide yes)
 			(show_name no)
@@
 	(symbol
 		(lib_id "Device:C_Polarized")
-		(at 209.55 35.56 0)
+		(at 203.2 35.56 0)
 		(unit 1)
 		(body_style 1)
@@
 		(fields_autoplaced yes)
 		(property "Reference" "C1"
-			(at 213.36 33.4009 0)
+			(at 207.01 33.4009 0)
 			(show_name no)
 			(do_not_autoplace no)
@@
 		)
 		(property "Value" "C_Polarized"
-			(at 213.36 35.9409 0)
+			(at 207.01 35.9409 0)
 			(show_name no)
 			(do_not_autoplace no)
@@
 		)
 		(property "Footprint" "Capacitor_THT:CP_Radial_D10.0mm_P3.50mm"
-			(at 210.5152 39.37 0)
+			(at 204.1652 39.37 0)
 			(hide yes)
 			(show_name no)
@@
 		)
 		(property "Datasheet" ""
-			(at 209.55 35.56 0)
+			(at 203.2 35.56 0)
 			(hide yes)
 			(show_name no)
@@
 		)
 		(property "Description" "Polarized capacitor"
-			(at 209.55 35.56 0)
+			(at 203.2 35.56 0)
 			(hide yes)
 			(show_name no)
@@
 	(symbol
 		(lib_id "power:GND")
-		(at 203.2 39.37 0)
+		(at 196.85 39.37 0)
 		(unit 1)
 		(body_style 1)
@@
 		(fields_autoplaced yes)
 		(property "Reference" "#PWR010"
-			(at 203.2 45.72 0)
+			(at 196.85 45.72 0)
 			(hide yes)
 			(show_name no)
@@
 		)
 		(property "Value" "GND"
-			(at 203.2 44.45 0)
+			(at 196.85 44.45 0)
 			(show_name no)
 			(do_not_autoplace no)
@@
 		)
 		(property "Footprint" ""
-			(at 203.2 39.37 0)
+			(at 196.85 39.37 0)
 			(hide yes)
 			(show_name no)
@@
 		)
 		(property "Datasheet" ""
-			(at 203.2 39.37 0)
+			(at 196.85 39.37 0)
 			(hide yes)
 			(show_name no)
@@
 		)
 		(property "Description" "Power symbol creates a global label with name \"GND\" , ground"
-			(at 203.2 39.37 0)
+			(at 196.85 39.37 0)
 			(hide yes)
 			(show_name no)
