File: nav_system.kicad_pcb (KiCad board)
At the start: 2 copper layers, 140 x 81 mm, 14 parts, among them J1 GPS MODULE, J10 SW-420, J2 MPU6050, J3 SIM76003-L1C, J4 ESP32-CAM, J5 SW-420, J6 MAIN POWER, J8 RGB, J9 RGB_GROUND

Commit message: Nav_system.2.0
Parts:
- added J7: DC FAN, Connector_JST:JST_XH_B2B-XH-A_1x02_P2.50mm_Vertical, F.Cu at (87.0, 120.0)
- J1: value GPS MODULE -> gps module; footprint Connector_PinSocket_2.54mm:PinSocket_1x04_P2.54mm_Vertical -> Connector_PinHeader_2.54mm:PinHeader_1x05_P2.54mm_Vertical
- J10: value SW-420 -> toggle
- J5: footprint Connector_JST:JST_XH_B3B-XH-A_1x03_P2.50mm_Vertical -> Connector_PinSocket_2.54mm:PinSocket_1x03_P2.54mm_Vertical; moved to B.Cu
- moved J2 85.9 mm to (95.9, 110.0), turned to -90 degrees
- moved J3 79.9 mm to (79.9, 55.0), turned to 90 degrees
- moved C1 72.5 mm to (182.5, 59.5)
- moved J6 56.8 mm to (181.5, 112.5)
- moved J8 53.6 mm to (169.5, 110.0), turned to -90 degrees
- moved U1 52.8 mm to (139.1, 115.5), turned to 180 degrees
- moved J10 46.5 mm to (122.5, 123.0)
- moved J9 46.0 mm to (158.5, 115.0), turned to 90 degrees
- moved J4 44.8 mm to (169.2, 57.5)
- moved R3 24.2 mm to (151.0, 101.2), turned to 180 degrees
- moved R1 24.2 mm to (151.0, 94.8), turned to 180 degrees
- moved R2 24.2 mm to (151.0, 98.0), turned to 180 degrees
- moved J1 7.26 mm to (162.8, 81.8)
- moved J5 4.34 mm to (145.0, 58.5)
Connections:
- J1 pad 1: GND -> unconnected-(J1-Pin_1-Pad1)
- J1 pad 2: /TX -> /RX
- J1 pad 3: /RX -> /TX
- J1 pad 4: VCC -> GND
- J3 pad 2: /RXD -> /TXD
- J3 pad 3: /TXD -> /RXD
- J5 pad 1: GND -> /DO
- J5 pad 2: /DO -> GND
Routing:
- net VCC: track 0.00 -> 151.2 mm
- net /RX: track 0.00 -> 84.4 mm
- net /DO: track 0.00 -> 73.8 mm
- net +3.3V: track 0.00 -> 71.8 mm
- net /TX: track 0.00 -> 70.3 mm
- net /TXD: track 0.00 -> 64.4 mm
- net /RXD: track 0.00 -> 60.1 mm
- net /PWRKEY: track 0.00 -> 51.7 mm
- net /g5: track 0.00 -> 35.8 mm
- net /SCL: track 0.00 -> 34.9 mm
- net /SDA: track 0.00 -> 32.3 mm
- net Net-(J8-Pin_1): track 0.00 -> 24.7 mm
- net Net-(J8-Pin_2): track 0.00 -> 24.5 mm
- net Net-(J8-Pin_3): track 0.00 -> 24.2 mm
- net /GREEN: track 0.00 -> 9.31 mm
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- added copper zone on B.Cu, net GND

Commit message: modify plot files
Parts:
- added J11: MAIN P SWITCH, Connector_JST:JST_XH_B2B-XH-A_1x02_P2.50mm_Vertical, F.Cu at (192.9, 98.0)
- moved J7 62.5 mm to (149.5, 120.5), turned to 180 degrees
- moved J3 7.03 mm to (80.5, 62.0)
- moved C1 0.12 mm to (182.5, 59.4), turned to -90 degrees
Connections:
- J6 pad 2: VCC -> Net-(J11-Pin_1)
Routing:
- net VCC: track 151.2 -> 300.3 mm
- net Net-(J11-Pin_1): track 0.00 -> 18.2 mm
- net +3.3V: track 71.8 -> 76.7 mm
- net /PWRKEY: track 51.7 -> 55.3 mm
- net /TX: track 70.3 -> 72.9 mm
- net /RXD: track 60.1 -> 57.7 mm
- net /SCL: track 34.9 -> 32.8 mm
- net /TXD: track 64.4 -> 62.9 mm

Commit message: update symbols
Parts:
- moved U1 0.20 mm to (139.0, 115.6)
Routing:
- net /TX: track 72.9 -> 81.5 mm
- net /RX: track 84.4 -> 89.9 mm
- net /TXD: track 62.9 -> 64.5 mm
- net /SCL: track 32.8 -> 34.4 mm
- net +3.3V: track 76.7 -> 75.5 mm
- net /GREEN: track 9.31 -> 10.5 mm
- net /DO: track 73.8 -> 72.7 mm
- net /SDA: track 32.3 -> 33.2 mm
- net /RXD: track 57.7 -> 58.6 mm
- net /PWRKEY: track 55.3 -> 56.2 mm
